File: PCB Files/rudyb2_kombucha_sensor+relay.kicad_pcb (KiCad board)
At the start: 2 copper layers, 97 x 93 mm, 47 parts, among them J1 Screw_Terminal_01x02, J10 Relay, J11 L298N, J13 ESP32 R, J2 ESP32 L, J3 Ultrasonic 1, J4 Ultrasonic 2, J5 Ultrasonic 3, J6 pH sensor, J7 RGB Sensor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

Commit message: Add files via upload
Parts:
- removed C4: 10 uF, Capacitor_SMD:C_0805_2012Metric_Pad1.18x1.45mm_HandSolder
- removed C5, C6: 0.1 uF, Capacitor_SMD:C_0805_2012Metric_Pad1.18x1.45mm_HandSolder
- removed R5, R6: 4.7k, Resistor_SMD:R_0805_2012Metric_Pad1.20x1.40mm_HandSolder
- removed U2: AMS1117-3.3, Package_TO_SOT_SMD:SOT-223-3_TabPin2
- added J12: Screw_Terminal_01x02, TerminalBlock:TerminalBlock_Xinya_XY308-2.54-2P_1x02_P2.54mm_Horizontal, F.Cu at (165.7, 58.6)
- added J14: Screw_Terminal_01x02, TerminalBlock:TerminalBlock_Xinya_XY308-2.54-2P_1x02_P2.54mm_Horizontal, F.Cu at (135.2, 139.8)
- added J15: Screw_Terminal_01x02, TerminalBlock:TerminalBlock_Xinya_XY308-2.54-2P_1x02_P2.54mm_Horizontal, F.Cu at (143.5, 140.0)
- added J16: Screw_Terminal_01x02, TerminalBlock:TerminalBlock_Xinya_XY308-2.54-2P_1x02_P2.54mm_Horizontal, F.Cu at (186.2, 138.4)
- added U1: AZ1117CD-3.3TRG1, AZ1117CD-3.3TRG1:DPAK457P1010X238-3N, F.Cu at (189.8, 57.9)
- moved TP6 19.7 mm to (210.5, 127.7)
- moved C7 14.2 mm to (201.9, 62.0), turned to 90 degrees
- moved TP3 12.0 mm to (193.3, 129.3)
- moved TP5 11.4 mm to (193.8, 124.2)
- moved TP9 10.3 mm to (207.1, 131.3)
- moved R7 8.58 mm to (168.7, 78.0)
- moved J9 7.21 mm to (154.2, 140.4)
- moved TP8 6.59 mm to (200.0, 129.4)
- moved TP4 6.28 mm to (188.6, 124.2)
- moved TP2 5.93 mm to (187.9, 129.6)
- moved C3 4.96 mm to (161.7, 69.3)
- moved TP7 1.26 mm to (200.1, 124.3)
- turned R12 to -90 degrees
Connections:
- C3 pad 2: Net-(U2-VI) -> GND
- C7 pad 1: Net-(U2-VO) -> +3.3V
- C7 pad 2: +3.3V -> GND
- J8 pad 1: Net-(J8-Pin_1) -> +3.3V
- R11 pad 1: /G19 -> GND
- R11 pad 2: /ECHO3 -> /G19
- R12 pad 1: /G35 -> GND
- R12 pad 2: /PH_OUT -> /G35
- R4 pad 1: /G17 -> GND
- R4 pad 2: /ECHO1 -> /G17
- R7 pad 1: +3.3V -> /DATA
- R7 pad 2: Net-(J8-Pin_1) -> +3.3V
- R9 pad 1: /G18 -> GND
- R9 pad 2: /ECHO2 -> /G18
Routing:
- net GND: track 22.8 -> 416.7 mm, vias 15 -> 20
- net +12V: track 0.00 -> 167.6 mm, vias 0 -> 2
- net Net-(J8-Pin_1): track 48.5 -> 0.00 mm, vias 4 -> 0
- net /ECHO3: track 108.3 -> 69.8 mm, vias 2 -> 4
- net /SCL: track 178.5 -> 140.8 mm, vias 8 -> 11
- net Net-(U2-VO): track 36.7 -> 0.00 mm
- net +3.3V: track 203.6 -> 237.1 mm, vias 4 -> 6
- net /DATA: track 118.0 -> 149.3 mm, vias 11 -> 10
- net Net-(U2-VI): track 23.7 -> 0.00 mm, vias 2 -> 0
- net +5V: track 353.3 -> 373.6 mm, vias 0 -> 2
- net /SDA: track 168.8 -> 153.8 mm
- net /ECHO2: track 61.4 -> 54.9 mm, vias 2 -> 4
- net /PH_OUT: track 130.4 -> 126.1 mm
- net /G18: track 36.9 -> 39.3 mm
- net /G35: track 64.8 -> 66.3 mm
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Other:
- board text added: "Team 27 Board v5.0 04/14/26"
- board text removed: "Team 27 Board v1.0 02/25/26"
