File: PCB Files/rudyb2_kombucha_sensor+relay.kicad_sch (KiCad schematic)
At the start: 47 parts, among them J1 Screw_Terminal_01x02, J10 Relay, J11 L298N, J13 ESP32 R, J2 ESP32 L, J3 Ultrasonic 1, J4 Ultrasonic 2, J5 Ultrasonic 3, J6 pH sensor, J7 RGB Sensor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

Commit message: Add files via upload
Parts:
- removed C4: 10 uF, Capacitor_SMD:C_0805_2012Metric_Pad1.18x1.45mm_HandSolder, symbol Device:C
- removed C5, C6: 0.1 uF, Capacitor_SMD:C_0805_2012Metric_Pad1.18x1.45mm_HandSolder, symbol Device:C
- removed R5, R6: 4.7k, Resistor_SMD:R_0805_2012Metric_Pad1.20x1.40mm_HandSolder, symbol Device:R
- removed U2: AMS1117-3.3, Package_TO_SOT_SMD:SOT-223-3_TabPin2, symbol Regulator_Linear:AMS1117-3.3
- added J12, J14, J15, J16: Screw_Terminal_01x02, TerminalBlock:TerminalBlock_Xinya_XY308-2.54-2P_1x02_P2.54mm_Horizontal, symbol Connector:Screw_Terminal_01x02
- added U1: AZ1117CD-3.3TRG1, AZ1117CD-3.3TRG1:DPAK457P1010X238-3N, symbol AZ11117CD:AZ1117CD-3.3TRG1
Connections:
- net +3.3V: now also C7.1, J8.1 (Pin_1), R7.2, U1.2 (OUTPUT); no longer C7.2, R7.1
- net +5V: now also U1.3 (INPUT)
- net DATA: now also R7.1
- net ECHO1: no longer R4.2
- net ECHO2: no longer R9.2
- net ECHO3: no longer R11.2
- net G17: now also R4.2; no longer R4.1
- net G18: now also R9.2; no longer R9.1
- net G19: now also R11.2; no longer R11.1
- net G35: now also R12.2; no longer R12.1
- net GND: now also C3.2, C7.2, R11.1, R12.1, R4.1, R9.1, J12.1 (Pin_1), J14.1 (Pin_1), J15.1 (Pin_1), J16.1 (Pin_1), U1.1 (ADJ/GND)
- net PH_OUT: no longer R12.2
- new net +12V: J12.2 (Pin_2), J14.2 (Pin_2), J15.2 (Pin_2), J16.2 (Pin_2)
Other:
- note added: "Team 27 Board v5.0 04/14/26"
- note removed: "Team 27 Board v1.0 02/20/26"
- moved on the sheet: C3, C7, R11, R7, R9, TP10
